File: Designs/LED_DRIVER_1/LED_DRIVER_1.sch (KiCad schematic (older format))
At the start: 1 part

Commit message: Working update
Parts:
- added C?: CP, symbol Device:CP
Connections:
- net 24V: now also U?.3 (VIN), C?.1; no longer U?.5 (PWM)
- net GND: now also C?.2
Changed lines of the file:
@@
 Wire Wire Line
 	5050 2650 5050 2800
-Text Label 3150 2150 0    50   ~ 0
+Text Label 2050 2250 0    50   ~ 0
 24V
+$Comp
+L power:GND #PWR?
+U 1 1 61014A91
+P 2350 3000
+F 0 "#PWR?" H 2350 2750 50  0001 C CNN
+F 1 "GND" H 2355 2827 50  0000 C CNN
+F 2 "" H 2350 3000 50  0001 C CNN
+F 3 "" H 2350 3000 50  0001 C CNN
+	1    2350 3000
+	1    0    0    -1
+$EndComp
 Wire Wire Line
-	3550 2150 3150 2150
+	2350 2850 2350 3000
+$Comp
+L Device:CP C?
+U 1 1 61014181
+P 2350 2700
+F 0 "C?" H 2468 2746 50  0000 L CNN
+F 1 "CP" H 2468 2655 50  0000 L CNN
+F 2 "" H 2388 2550 50  0001 C CNN
+F 3 "~" H 2350 2700 50  0001 C CNN
+	1    2350 2700
+	1    0    0    -1
+$EndComp
+Wire Wire Line
+	2050 2250 2350 2250
+Wire Wire Line
+	2350 2550 2350 2250
+Connection ~ 2350 2250
+Wire Wire Line
+	2350 2250 3550 2250
 $EndSCHEMATC
